File: NoisyBoi.kicad_pcb (KiCad board)
At the start: 2 copper layers, 85 x 82.5 mm, 36 parts, among them U1 OPA2134UA

Commit message: update
Connections:
- net +4.5V renamed V-+
- net -4.5V renamed V--

Commit message: fix typo (damnit)
Parts:
- removed kibuzzard-691D64F6 (x2): G***, kibuzzard-691D64F6
- removed kibuzzard-691D65D8 (x2): G***, kibuzzard-691D65D8
- added kibuzzard-691D6DA0: G***, kibuzzard-691D6DA0, B.Cu at (142.0, 72.8)
- added kibuzzard-691D6DA7: G***, kibuzzard-691D6DA7, B.Cu at (142.0, 72.8)
- added kibuzzard-691D6DFD: G***, kibuzzard-691D6DFD, F.Cu at (142.0, 72.8)
- added kibuzzard-691D6E02: G***, kibuzzard-691D6E02, F.Cu at (142.0, 72.8)
- moved kibuzzard-691D6368 0.69 mm to (141.6, 62.0) (x2)
- moved kibuzzard-691D6378 0.69 mm to (141.6, 62.0) (x2)
- moved kibuzzard-691D6399 0.38 mm to (141.7, 67.3) (x2)
- moved kibuzzard-691D639E 0.38 mm to (141.7, 67.3) (x2)
